Commit message: Update project (README and package files)

File: src/my_robot_description/urdf/mobile_base.xacro (robot description, xacro)
@@ -58,6 +58,5 @@
     <xacro:sphere_inertia m="0.5" r="${2.0*wheel_radius * 0.5}" xyz="0 0 0" rpy="0 0 0"/>
   </link>
-  <link name="base_footprint">
-  </link>
+  <link name="base_footprint" />
   <joint name="base_right_wheel_joint" type="continuous">
     <parent link="base_link"/>

File: src/my_robot_description/urdf/mobile_base_gazebo.xacro (robot description, xacro)
@@ -12,4 +12,25 @@
   <gazebo reference="caster_wheel_link">
     <material>Gazebo/Grey</material>
+    <mu1 value="0.1"/>
+    <mu2 value="0.1"/>
+  </gazebo>
+  <gazebo>
+   <!-- plugin name changed to avoid multiple ROS nodes with same name -->
+   <plugin name="my_robot_diff_drive" filename="libgazebo_ros_diff_drive.so">
+      <!-- explicitly assign a ROS node name to avoid collisions -->
+      <node_name>my_robot_diff_drive</node_name>
+      <update_rate>50</update_rate>
+      <left_joint>base_left_wheel_joint</left_joint>
+      <right_joint>base_right_wheel_joint</right_joint>
+      <wheel_separation>0.45</wheel_separation>
+      <wheel_diameter>0.2</wheel_diameter>
+      <command_topic>cmd_vel</command_topic>
+      <odometry_topic>odom</odometry_topic>
+      <odometry_frame>odom</odometry_frame>
+      <robot_base_frame>base_footprint</robot_base_frame>
+      <publish_odom>true</publish_odom>
+      <publish_odom_tf>true</publish_odom_tf>
+      <publish_wheel_tf>true</publish_wheel_tf>
+   </plugin>
   </gazebo>
 </robot>

File: src/my_robot_description/urdf/my_robot.urdf.xacro (robot description, xacro)
@@ -4,3 +4,4 @@
   <xacro:include filename="mobile_base.xacro"/>
   <xacro:include filename="mobile_base_gazebo.xacro"/>
+  <xacro:include filename="camera.xacro"/>
 </robot>
